File: led-board/led-board.kicad_pcb (KiCad board)
At the start: 2 copper layers, 0 parts

Commit message: Finalized Rev-1.0
Parts:
- added D1: LED, LED_THT:LED_D3.0mm, F.Cu at (56.5, 29.8)
- added D10: LED, LED_THT:LED_D3.0mm, F.Cu at (64.1, 37.5)
- added D11: LED, LED_THT:LED_D3.0mm, F.Cu at (71.8, 37.5)
- added D12: LED, LED_THT:LED_D3.0mm, F.Cu at (79.4, 37.5)
- added D13: LED, LED_THT:LED_D3.0mm, F.Cu at (87.0, 37.5)
- added D14: LED, LED_THT:LED_D3.0mm, F.Cu at (94.6, 37.5)
- added D15: LED, LED_THT:LED_D3.0mm, F.Cu at (102.2, 37.5)
- added D16: LED, LED_THT:LED_D3.0mm, F.Cu at (109.9, 37.5)
- added D17: LED, LED_THT:LED_D3.0mm, F.Cu at (56.5, 45.1)
- added D18: LED, LED_THT:LED_D3.0mm, F.Cu at (64.1, 45.1)
- added D19: LED, LED_THT:LED_D3.0mm, F.Cu at (71.8, 45.1)
- added D2: LED, LED_THT:LED_D3.0mm, F.Cu at (64.1, 29.8)
- added D20: LED, LED_THT:LED_D3.0mm, F.Cu at (79.4, 45.1)
- added D21: LED, LED_THT:LED_D3.0mm, F.Cu at (87.0, 45.1)
- added D22: LED, LED_THT:LED_D3.0mm, F.Cu at (94.6, 45.1)
- added D23: LED, LED_THT:LED_D3.0mm, F.Cu at (102.2, 45.1)
- added D24: LED, LED_THT:LED_D3.0mm, F.Cu at (109.9, 45.1)
- added D25: LED, LED_THT:LED_D3.0mm, F.Cu at (56.5, 52.7)
- added D26: LED, LED_THT:LED_D3.0mm, F.Cu at (64.1, 52.7)
- added D27: LED, LED_THT:LED_D3.0mm, F.Cu at (71.8, 52.7)
- added D28: LED, LED_THT:LED_D3.0mm, F.Cu at (79.4, 52.7)
- added D29: LED, LED_THT:LED_D3.0mm, F.Cu at (87.0, 52.7)
- added D3: LED, LED_THT:LED_D3.0mm, F.Cu at (71.8, 29.8)
- added D30: LED, LED_THT:LED_D3.0mm, F.Cu at (94.6, 52.7)
- added D31: LED, LED_THT:LED_D3.0mm, F.Cu at (102.2, 52.7)
- added D32: LED, LED_THT:LED_D3.0mm, F.Cu at (109.9, 52.7)
- added D33: LED, LED_THT:LED_D3.0mm, F.Cu at (56.5, 60.3)
- added D34: LED, LED_THT:LED_D3.0mm, F.Cu at (64.1, 60.3)
- added D35: LED, LED_THT:LED_D3.0mm, F.Cu at (71.7, 60.3)
- added D36: LED, LED_THT:LED_D3.0mm, F.Cu at (79.3, 60.3)
- added D37: LED, LED_THT:LED_D3.0mm, F.Cu at (87.0, 60.3)
- added D38: LED, LED_THT:LED_D3.0mm, F.Cu at (94.6, 60.3)
- added D39: LED, LED_THT:LED_D3.0mm, F.Cu at (102.2, 60.3)
- added D4: LED, LED_THT:LED_D3.0mm, F.Cu at (79.4, 29.8)
- added D40: LED, LED_THT:LED_D3.0mm, F.Cu at (109.8, 60.3)
- added D41: LED, LED_THT:LED_D3.0mm, F.Cu at (56.5, 67.9)
- added D42: LED, LED_THT:LED_D3.0mm, F.Cu at (64.1, 67.9)
- added D43: LED, LED_THT:LED_D3.0mm, F.Cu at (71.8, 67.9)
- added D44: LED, LED_THT:LED_D3.0mm, F.Cu at (79.4, 67.9)
- added D45: LED, LED_THT:LED_D3.0mm, F.Cu at (87.0, 67.9)
- added D46: LED, LED_THT:LED_D3.0mm, F.Cu at (94.6, 67.9)
- added D47: LED, LED_THT:LED_D3.0mm, F.Cu at (102.2, 67.9)
- added D48: LED, LED_THT:LED_D3.0mm, F.Cu at (109.9, 67.9)
- added D49: LED, LED_THT:LED_D3.0mm, F.Cu at (56.5, 75.6)
- added D5: LED, LED_THT:LED_D3.0mm, F.Cu at (87.0, 29.8)
- added D50: LED, LED_THT:LED_D3.0mm, F.Cu at (64.1, 75.6)
- added D51: LED, LED_THT:LED_D3.0mm, F.Cu at (71.7, 75.6)
- added D52: LED, LED_THT:LED_D3.0mm, F.Cu at (79.3, 75.6)
- added D53: LED, LED_THT:LED_D3.0mm, F.Cu at (87.0, 75.6)
- added D54: LED, LED_THT:LED_D3.0mm, F.Cu at (94.6, 75.6)
- added D55: LED, LED_THT:LED_D3.0mm, F.Cu at (102.2, 75.6)
- added D56: LED, LED_THT:LED_D3.0mm, F.Cu at (109.8, 75.6)
- added D57: LED, LED_THT:LED_D3.0mm, F.Cu at (56.5, 83.2)
- added D58: LED, LED_THT:LED_D3.0mm, F.Cu at (64.1, 83.2)
- added D59: LED, LED_THT:LED_D3.0mm, F.Cu at (71.8, 83.2)
- added D6: LED, LED_THT:LED_D3.0mm, F.Cu at (94.6, 29.8)
- added D60: LED, LED_THT:LED_D3.0mm, F.Cu at (79.4, 83.2)
- added D61: LED, LED_THT:LED_D3.0mm, F.Cu at (87.0, 83.2)
- added D62: LED, LED_THT:LED_D3.0mm, F.Cu at (94.6, 83.2)
- added D63: LED, LED_THT:LED_D3.0mm, F.Cu at (102.2, 83.2)
- added D64: LED, LED_THT:LED_D3.0mm, F.Cu at (109.9, 83.2)
- added D7: LED, LED_THT:LED_D3.0mm, F.Cu at (102.2, 29.8)
- added D8: LED, LED_THT:LED_D3.0mm, F.Cu at (109.9, 29.8)
- added D9: LED, LED_THT:LED_D3.0mm, F.Cu at (56.5, 37.5)
- added FID1: 1mm, Fiducial:Fiducial_1mm_Mask2mm, F.Cu at (50.8, 28.6)
- added FID2: 1mm, Fiducial:Fiducial_1mm_Mask2mm, F.Cu at (115.6, 28.6)
- added FID3: 1mm, Fiducial:Fiducial_1mm_Mask2mm, F.Cu at (100.3, 93.3)
- added J1: Conn_02x08_Odd_Even, Connector_PinHeader_2.54mm:PinHeader_2x08_P2.54mm_Horizontal, B.Cu at (74.3, 90.8)
- added MH1: M3, MountingHole:MountingHole_2.2mm_M2_DIN965_Pad, F.Cu at (52.1, 24.1)
- added MH2: M3, MountingHole:MountingHole_2.2mm_M2_DIN965_Pad, F.Cu at (114.3, 24.1)
- added MH3: M3, MountingHole:MountingHole_2.2mm_M2_DIN965_Pad, F.Cu at (52.1, 94.0)
- added MH4: M3, MountingHole:MountingHole_2.2mm_M2_DIN965_Pad, F.Cu at (114.3, 94.0)
- added TP1: TestPoint, TestPoint:TestPoint_Pad_D1.0mm, F.Cu at (56.5, 24.1)
- added TP10: TestPoint, TestPoint:TestPoint_Pad_D1.0mm, F.Cu at (63.0, 92.3)
- added TP2: TestPoint, TestPoint:TestPoint_Pad_D1.0mm, F.Cu at (64.1, 24.1)
- added TP3: TestPoint, TestPoint:TestPoint_Pad_D1.0mm, F.Cu at (71.8, 24.1)
- added TP4: TestPoint, TestPoint:TestPoint_Pad_D1.0mm, F.Cu at (79.4, 24.1)
- added TP5: TestPoint, TestPoint:TestPoint_Pad_D1.0mm, F.Cu at (87.0, 24.1)
- added TP6: TestPoint, TestPoint:TestPoint_Pad_D1.0mm, F.Cu at (94.6, 24.1)
- added TP7: TestPoint, TestPoint:TestPoint_Pad_D1.0mm, F.Cu at (102.2, 24.1)
- added TP8: TestPoint, TestPoint:TestPoint_Pad_D1.0mm, F.Cu at (109.9, 24.1)
Routing:
- net /Row1: track 0.00 -> 134.0 mm, vias 0 -> 1
- net /Row2: track 0.00 -> 132.7 mm
- net /Row3: track 0.00 -> 121.0 mm, vias 0 -> 1
- net /Row5: track 0.00 -> 116.6 mm
- net /Row4: track 0.00 -> 113.5 mm, vias 0 -> 1
- net /Row6: track 0.00 -> 101.6 mm
- net /Led8: track 0.00 -> 99.5 mm, vias 0 -> 1
- net /Led1: track 0.00 -> 98.4 mm
- net /Led2: track 0.00 -> 95.2 mm, vias 0 -> 1
- net /Led7: track 0.00 -> 93.3 mm, vias 0 -> 1
- net /Led3: track 0.00 -> 90.7 mm, vias 0 -> 1
- net /Led6: track 0.00 -> 87.7 mm, vias 0 -> 1
- net /Led4: track 0.00 -> 86.8 mm, vias 0 -> 1
- net /Led5: track 0.00 -> 83.7 mm, vias 0 -> 1
- net /Row7: track 0.00 -> 82.8 mm
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- added copper zone on B.Cu, net GND
- added copper zone on F.Cu, net GND
Other:
- board outline added: 68.6 x 76.5 mm
- board text added: "JLCJLCJLCJLC"
- board text removed: "Tips: - Minimum grid : 0.25mm - Theme: Monokai High Contrast"
