File: led-board/led-board.kicad_sch (KiCad schematic)
At the start: 72 parts, among them J1 Conn_02x08_Odd_Even

Commit message: Finalized Rev-1.0
Parts:
- added TP1, TP10, TP2, TP3, TP4, TP5, TP6, TP7, TP8: TestPoint, TestPoint:TestPoint_Pad_D1.0mm, symbol Connector:TestPoint
- D1, D10, D11, D12, D13, D14, D15, D16, D17, D18, D19, D2, D20, D21, D22, D23, D24, D25, D26, D27, D28, D29, D3, D30, D31, D32, D33, D34, D35, D36, D37, D38, D39, D4, D40, D41, D42, D43, D44, D45, D46, D47, D48, D49, D5, D50, D51, D52, D53, D54, D55, D56, D57, D58, D59, D6, D60, D61, D62, D63, D64, D7, D8, D9: footprint (none) -> LED_THT:LED_D3.0mm
- FID1, FID2, FID3: now not fitted
- J1: footprint (none) -> Connector_PinHeader_2.54mm:PinHeader_2x08_P2.54mm_Horizontal; now not fitted; now left out of the parts list
- MH1, MH2, MH3, MH4: footprint MountingHole:MountingHole_3.2mm_M3_Pad_Via -> MountingHole:MountingHole_2.2mm_M2_DIN965_Pad; now not fitted
Connections:
- net Led1: now also TP1.1
- net Led2: now also TP2.1
- net Led3: now also TP3.1
- net Led4: now also TP4.1
- net Led5: now also TP5.1
- net Led6: now also TP6.1
- net Led7: now also TP7.1; no longer D16.2 (A), D24.2 (A), D32.2 (A), D40.2 (A), D48.2 (A), D56.2 (A), D64.2 (A), D8.2 (A), J1.15 (Pin_15)
- net Row1: now also TP10.1
- net Row5: now also D34.1 (K), D35.1 (K), D36.1 (K), D37.1 (K), D38.1 (K), D39.1 (K)
- new net Led8: D16.2 (A), D24.2 (A), D32.2 (A), D40.2 (A), D48.2 (A), D56.2 (A), D64.2 (A), D8.2 (A), J1.15 (Pin_15), TP8.1
Other:
- note removed: "3 Fiducials/component-layer"

Commit message: led-board minor update
Parts:
- J1: now fitted
